File: ADM3260_Breakout.brd (EAGLE design)
At the start: 64.4 x 26.9 mm, 21 parts, among them J2 BNCPTH, Q1 PMV32UP, Q2 PMV16XN, Q3 PMV32UP, U1 ADM3260, U2 OEM EZO pH

Commit message: update
Parts:
- moved R3 2.93 mm to (128.1, 54.9), turned to 90 degrees
- moved C8 2.10 mm to (125.7, 51.5), turned to 0 degrees
- moved C5 1.06 mm to (121.8, 46.2)
- moved C6 0.91 mm to (123.8, 46.0)
- moved C7 0.64 mm to (123.8, 49.7), turned to 0 degrees
- moved R6 0.58 mm to (128.1, 45.2)
- moved R5 0.42 mm to (128.1, 49.1)
Routing:
- net 3V3-ISO: track 0.00 -> 22.1 mm, vias 0 -> 5
- net SDA1: track 22.1 -> 28.6 mm

Commit message: Update
Parts:
- moved R2 3.18 mm to (107.3, 53.4), turned to 90 degrees
- moved R1 2.42 mm to (105.5, 55.4), turned to 270 degrees
- moved C4 0.09 mm to (107.3, 49.8)
- moved C3 0.07 mm to (105.4, 49.7)
Connections:
- net GND: now also J1.4; no longer J1.5
- net VCC: now also J1.5; no longer J1.4
Routing:
- net AVCC: track 0.00 -> 18.0 mm, vias 0 -> 3
- net SCL2: track 14.7 -> 16.2 mm
- net SDA2: track 14.4 -> 13.0 mm
- net VCC: track 14.6 -> 13.2 mm
- net EN: track 12.1 -> 12.8 mm

Commit message: finished, but not checked for errors yet
Connections:
- net N$8 renamed PRB
Routing:
- net GND-ISO: track 0.00 -> 51.1 mm
- net 3V3-ISO: track 22.1 -> 23.4 mm
- added copper zone on layer 15, net 3V3-ISO
- added copper zone on layer 2, net AVCC
- added copper zone on layer 2, net BNC_PLANE_L2
- added copper zone on layer 15, net BNC_PLANE_L3
- added copper zone on layer 16, net BNC_PLANE_L4
- added copper zone on layer 15, net GND
- added copper zone on layer 16, net GND
- added copper zone on layer 16, net GND-ISO
- added copper zone on layer 2, net GND-ISO
- added copper zone on layer 15, net PRBGND
- added copper zone on layer 16, net PRBGND
- added copper zone on layer 2, net PRBGND

Commit message: update
Routing:
- net GND-ISO: track 51.1 -> 55.7 mm, vias 49 -> 42
- net EN: track 12.8 -> 15.8 mm
- net AVCC: track 18.0 -> 20.4 mm, vias 3 -> 4
- added copper zone on layer 1, net BNC_PLANE
- added copper zone on layer 15, net BNC_PLANE
- added copper zone on layer 16, net BNC_PLANE
- added copper zone on layer 2, net BNC_PLANE
- removed copper zone on layer 1, net BNC_PLANE_L1
- removed copper zone on layer 2, net BNC_PLANE_L2
- removed copper zone on layer 15, net BNC_PLANE_L3
- removed copper zone on layer 16, net BNC_PLANE_L4

Commit message: update
Routing:
- net GND-ISO: track 55.7 -> 0.00 mm
- net SDA1: track 28.6 -> 27.3 mm
- added copper zone on layer 15, net GND-ISO

Commit message: update
Parts:
- U2: value OEM EZO pH -> Atlas Scientific OEM pH or ORP
- moved R5 2.10 mm to (127.4, 47.2)
- moved R6 2.10 mm to (127.4, 43.2)
- moved C4 1.68 mm to (109.0, 49.7)
- moved C3 1.57 mm to (107.0, 49.7)
Routing:
- net GND-ISO: track 0.00 -> 55.1 mm
- net AVCC: track 20.6 -> 19.4 mm
- net N$1: track 11.0 -> 11.6 mm
- added copper zone on layer 3, net 3V3-ISO
- added copper zone on layer 3, net BNC_PLANE
- added copper zone on layer 3, net GND
- added copper zone on layer 3, net PRBGND
- removed copper zone on layer 15, net 3V3-ISO
- removed copper zone on layer 15, net BNC_PLANE
- removed copper zone on layer 15, net GND
- removed copper zone on layer 15, net GND-ISO
- removed copper zone on layer 15, net PRBGND
Other:
- board size 64.4 x 26.9 mm -> 63.8 x 26.4 mm
