File: ADM3260_Breakout.sch (EAGLE design)
At the start: 21 parts, among them J2 BNCPTH, Q1 PMV32UP, Q2 PMV16XN, Q3 PMV32UP, U1 ADM3260, U2 OEM EZO pH

Commit message: Update
Connections:
- net GND: now also J1.4; no longer J1.5
- net VCC: now also J1.5; no longer J1.4
Changed lines of the file:
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@@
 <part name="SUPPLY1" library="supply2" library_urn="urn:adsk.eagle:library:372" deviceset="GND" device="" value="GNDP"/>
 <part name="SUPPLY2" library="supply2" library_urn="urn:adsk.eagle:library:372" deviceset="GND" device="" value="GNDP"/>
-<part name="SUPPLY4" library="supply2" library_urn="urn:adsk.eagle:library:372" deviceset="GND" device="" value="GNDP"/>
 <part name="SUPPLY3" library="supply2" library_urn="urn:adsk.eagle:library:372" deviceset="GND" device="" value="GNDP"/>
 <part name="SUPPLY5" library="supply2" library_urn="urn:adsk.eagle:library:372" deviceset="GND" device="" value="GNDP"/>
+<part name="SUPPLY4" library="supply2" library_urn="urn:adsk.eagle:library:372" deviceset="GND" device="" value="GNDP"/>
 </parts>
 <sheets>
@@
 <attribute name="VALUE" x="-40.005" y="47.625" size="1.778" layer="96"/>
 </instance>
-<instance part="SUPPLY4" gate="GND" x="-99.06" y="76.2" smashed="yes">
-<attribute name="VALUE" x="-100.965" y="73.025" size="1.778" layer="96"/>
-</instance>
 <instance part="SUPPLY3" gate="GND" x="-58.42" y="76.2" smashed="yes">
 <attribute name="VALUE" x="-60.325" y="73.025" size="1.778" layer="96"/>
@@
 <instance part="SUPPLY5" gate="GND" x="-33.02" y="121.92" smashed="yes">
 <attribute name="VALUE" x="-34.925" y="118.745" size="1.778" layer="96"/>
+</instance>
+<instance part="SUPPLY4" gate="GND" x="-99.06" y="81.28" smashed="yes">
+<attribute name="VALUE" x="-100.965" y="78.105" size="1.778" layer="96"/>
 </instance>
 </instances>
@@
 </segment>
 <segment>
-<pinref part="J1" gate="G$1" pin="4"/>
-<wire x1="-91.44" y1="86.36" x2="-96.52" y2="86.36" width="0.1524" layer="91"/>
-<wire x1="-96.52" y1="86.36" x2="-96.52" y2="83.82" width="0.1524" layer="91"/>
-<wire x1="-96.52" y1="83.82" x2="-99.06" y2="83.82" width="0.1524" layer="91"/>
-<label x="-99.06" y="83.82" size="1.778" layer="95" rot="R180" xref="yes"/>
+<pinref part="J1" gate="G$1" pin="5"/>
+<wire x1="-91.44" y1="83.82" x2="-91.44" y2="73.66" width="0.1524" layer="91"/>
+<wire x1="-91.44" y1="73.66" x2="-99.06" y2="73.66" width="0.1524" layer="91"/>
+<label x="-99.06" y="73.66" size="1.778" layer="95" rot="R180" xref="yes"/>
 </segment>
 </net>
@@
 <wire x1="-38.1" y1="53.34" x2="-38.1" y2="55.88" width="0.1524" layer="91"/>
 <pinref part="SUPPLY2" gate="GND" pin="GND"/>
-</segment>
-<segment>
-<pinref part="J1" gate="G$1" pin="5"/>
-<wire x1="-91.44" y1="83.82" x2="-93.98" y2="83.82" width="0.1524" layer="91"/>
-<wire x1="-93.98" y1="83.82" x2="-93.98" y2="78.74" width="0.1524" layer="91"/>
-<wire x1="-93.98" y1="78.74" x2="-99.06" y2="78.74" width="0.1524" layer="91"/>
-<pinref part="SUPPLY4" gate="GND" pin="GND"/>
 </segment>
 <segment>
@@
 <wire x1="-58.42" y1="78.74" x2="-48.26" y2="78.74" width="0.1524" layer="91"/>
 </segment>
-</net>
+<segment>
+<pinref part="J1" gate="G$1" pin="4"/>
+<wire x1="-91.44" y1="86.36" x2="-96.52" y2="86.36" width="0.1524" layer="91"/>
+<wire x1="-96.52" y1="86.36" x2="-96.52" y2="83.82" width="0.1524" layer="91"/>
+<wire x1="-96.52" y1="83.82" x2="-99.06" y2="83.82" width="0.1524" layer="91"/>
+<pinref part="SUPPLY4" gate="GND" pin="GND"/>
+</segment>
+</net>

Commit message: finished, but not checked for errors yet
Connections:
- net N$8 renamed PRB
Changed lines of the file:
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@@
 </segment>
 </net>
-<net name="N$8" class="0">
+<net name="PRB" class="0">
 <segment>
 <pinref part="U2" gate="G$1" pin="PRB"/>

Commit message: update
Parts:
- U2: value OEM EZO pH -> Atlas Scientific OEM pH or ORP
Changed lines of the file:
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@@
 <part name="R6" library="SparkFun-Resistors" deviceset="10KOHM" device="-0603-1/10W-1%" value="10k"/>
 <part name="GND-ISO4" library="SparkFun-PowerSymbols" deviceset="GND-ISO" device=""/>
-<part name="U2" library="SENSOR" deviceset="PHSENSOR" device="" value="OEM EZO pH"/>
+<part name="U2" library="SENSOR" deviceset="PHSENSOR" device="" value="Atlas Scientific OEM pH or ORP"/>
 <part name="GND-ISO5" library="SparkFun-PowerSymbols" deviceset="GND-ISO" device=""/>
 <part name="J2" library="SparkFun-Connectors" deviceset="BNC" device="PTH"/>
@@
 <part name="SUPPLY5" library="supply2" library_urn="urn:adsk.eagle:library:372" deviceset="GND" device="" value="GNDP"/>
 <part name="SUPPLY4" library="supply2" library_urn="urn:adsk.eagle:library:372" deviceset="GND" device="" value="GNDP"/>
+<part name="FRAME1" library="SparkFun-Aesthetics" deviceset="FRAME-A4L" device="">
+<attribute name="CNAME" value="ADM3260 with Atlas Scientific OEM pH or ORP"/>
+<attribute name="CREVISION" value="1.0.0"/>
+<attribute name="DESIGNER" value="Igor Knippenberg"/>
+</part>
 </parts>
 <sheets>
@@
 </instance>
 <instance part="SUPPLY4" gate="GND" x="-99.06" y="81.28" smashed="yes">
-<attribute name="VALUE" x="-100.965" y="78.105" size="1.778" layer="96"/>
+<attribute name="VALUE" x="-104.521" y="77.089" size="2.54" layer="96"/>
+</instance>
+<instance part="FRAME1" gate="G$1" x="-142.24" y="-22.86" smashed="yes">
+<attribute name="LAST_DATE_TIME" x="39.37" y="-16.51" size="2.286" layer="94" font="vector"/>
+<attribute name="SHEET" x="53.34" y="-21.59" size="2.54" layer="94" font="vector"/>
+<attribute name="DESIGNER" x="101.8" y="-16.51" size="2.54" layer="94" font="vector"/>
+<attribute name="CNAME" x="39.37" y="-6.35" size="2.54" layer="94" font="vector"/>
+<attribute name="CREVISION" x="92.68" y="-21.69" size="2.54" layer="94" font="vector"/>
 </instance>
 </instances>
@@
 <pinref part="J1" gate="G$1" pin="3"/>
 <wire x1="-91.44" y1="88.9" x2="-99.06" y2="88.9" width="0.1524" layer="91"/>
-<label x="-99.06" y="88.9" size="1.778" layer="95" rot="R180" xref="yes"/>
+<label x="-99.06" y="88.9" size="2.54" layer="95" rot="R180" xref="yes"/>
 </segment>
 </net>
@@
 <wire x1="-91.44" y1="83.82" x2="-91.44" y2="73.66" width="0.1524" layer="91"/>
 <wire x1="-91.44" y1="73.66" x2="-99.06" y2="73.66" width="0.1524" layer="91"/>
-<label x="-99.06" y="73.66" size="1.778" layer="95" rot="R180" xref="yes"/>
+<label x="-99.06" y="73.66" size="2.54" layer="95" rot="R180" xref="yes"/>
 </segment>
 </net>
@@
 <wire x1="35.56" y1="132.08" x2="40.64" y2="132.08" width="0.1524" layer="91"/>
 <wire x1="35.56" y1="132.08" x2="35.56" y2="134.62" width="0.1524" layer="91"/>
-<label x="35.56" y="134.62" size="1.778" layer="95" rot="R90" xref="yes"/>
+<label x="35.56" y="134.62" size="2.54" layer="95" rot="R90" xref="yes"/>
 </segment>
 <segment>
@@
 <wire x1="38.1" y1="101.6" x2="48.26" y2="101.6" width="0.1524" layer="91"/>
 <junction x="38.1" y="101.6"/>
-<label x="48.26" y="101.6" size="1.778" layer="95" xref="yes"/>
+<label x="48.26" y="101.6" size="2.54" layer="95" xref="yes"/>
 </segment>
 <segment>
@@
 <wire x1="38.1" y1="63.5" x2="45.72" y2="63.5" width="0.1524" layer="91"/>
 <junction x="38.1" y="63.5"/>
-<label x="45.72" y="63.5" size="1.778" layer="95" xref="yes"/>
+<label x="45.72" y="63.5" size="2.54" layer="95" xref="yes"/>
 </segment>
 </net>
@@
 <wire x1="40.64" y1="116.84" x2="48.26" y2="116.84" width="0.1524" layer="91"/>
 <junction x="40.64" y="116.84"/>
-<label x="48.26" y="116.84" size="1.778" layer="95" xref="yes"/>
+<label x="48.26" y="116.84" size="2.54" layer="95" xref="yes"/>
 </segment>
 </net>
@@
 <wire x1="30.48" y1="109.22" x2="48.26" y2="109.22" width="0.1524" layer="91"/>
 <junction x="30.48" y="109.22"/>
-<label x="48.26" y="109.22" size="1.778" layer="95" xref="yes"/>
-</segment>
-</net>
+<label x="48.26" y="109.22" size="2.54" layer="95" xref="yes"/>
+</segment>
+</net>
